Commit message: cleanup model

File: urdf/table.urdf.xacro (robot description, xacro)
@@ -13,9 +13,9 @@
        xmlns:controller="http://playerstage.sourceforge.net/gazebo/xmlschema/#controller"
        xmlns:physics="http://playerstage.sourceforge.net/gazebo/xmlschema/#physics">
-  <property name="table_height" value="0.8" />
+  <property name="table_height" value="0.92" />
   <property name="table_width" value="1.525" />
   <property name="table_depth" value=".760" />
   <property name="leg_radius" value="0.02" />
-  <property name="table_x" value="0.98" />
+  <property name="table_x" value="0.0" />
   <property name="table_y" value="0.0" />
   <property name="table_z" value="0.0" />
@@ -25,9 +25,9 @@
   <link name="table_top_link">
     <inertial>
-      <mass value="1.0" />
+      <mass value="1000.0" />
       <origin xyz="${table_x} ${table_y} ${table_z+table_height-table_top_thickness/2}" />
-      <inertia ixx="1" ixy="0"  ixz="0"
-               iyy="1" iyz="0"
-               izz="1" />
+      <inertia ixx="1000" ixy="0"  ixz="0"
+               iyy="1000" iyz="0"
+               izz="1000" />
     </inertial>
     <visual>

File: urdf/ur5_robotiq_joint_limited_robot.urdf.xacro (robot description, xacro)
@@ -3,13 +3,13 @@
 <!-- common stuff -->
 <xacro:include filename="$(find ur_description)/urdf/common.gazebo.xacro" />
-  <!-- ur5 -->
-  <xacro:include filename="$(find ur_description)/urdf/ur5.urdf.xacro" />
+<!-- ur5 -->
+<xacro:include filename="$(find ur_description)/urdf/ur5.urdf.xacro" />
  <!-- table leg  to world-->
-  <link name="world" />
-  <joint name="world_joint" type="fixed">
+  <!--link name="world" /-->
+  <!--joint name="world_joint" type="fixed">
     <parent link="world" />
     <child link = "table_top_link" />
     <origin rpy="0.0 0.0 0.0" xyz="0.0 0.0 0.0" />
-  </joint>
+  </joint-->
   <!-- arm top table-->
 <xacro:include filename="$(find manipulator_description)/urdf/table.urdf.xacro" />
@@ -17,5 +17,5 @@
     <parent link="table_top_link" />
     <child link = "base_link" />
-    <origin xyz="${table_x} ${table_y} ${table_z+table_height}" rpy="0.0 0.1 0.0" />
+    <origin xyz="${table_x} -0.21 ${table_height+0.005}" rpy="0.0 0.0 0.0" />
   </joint>
   <xacro:ur5_robot prefix="" joint_limited="true"/>
