Commit message: Mods:28022018

File: urdf/ur5_robotiq_joint_limited_robot.urdf.xacro (robot description, xacro)
@@ -3,5 +3,5 @@
 <robot xmlns:xacro="http://www.ros.org/wiki/xacro" name="ur5">
   <!-- common stuff -->
-  <!--xacro:include filename="$(find ur_description)/urdf/common.gazebo.xacro" /-->
+  <xacro:include filename="$(find ur_description)/urdf/common.gazebo.xacro" />
   <!-- ur5 -->
   <xacro:include filename="$(find ur_description)/urdf/ur5.urdf.xacro" />
@@ -11,5 +11,5 @@
     <parent link="world" />
     <child link = "base_link" />
-    <origin rpy="0.0 0.0 0.0" xyz="0.04 0.46 0.8" />
+    <origin rpy="0.0 0.0 0.0" xyz="0.0 0.0 0.0" />
   </joint>
   <xacro:ur5_robot prefix="" joint_limited="true"/>

Commit message: Table stuff

File: urdf/ur5_robotiq_joint_limited_robot.urdf.xacro (robot description, xacro)
@@ -1,18 +1,24 @@
 <?xml version="1.0"?>
-<!--robot xmlns:xacro="http://www.ros.org/wiki/xacro" name="ur5"-->
 <robot xmlns:xacro="http://www.ros.org/wiki/xacro" name="ur5">
-  <!-- common stuff -->
-  <xacro:include filename="$(find ur_description)/urdf/common.gazebo.xacro" />
+<!-- common stuff -->
+<xacro:include filename="$(find ur_description)/urdf/common.gazebo.xacro" />
   <!-- ur5 -->
   <xacro:include filename="$(find ur_description)/urdf/ur5.urdf.xacro" />
-  <!-- arm -->
+ <!-- table leg  to world-->
   <link name="world" />
   <joint name="world_joint" type="fixed">
     <parent link="world" />
-    <child link = "base_link" />
+    <child link = "table_top_link" />
     <origin rpy="0.0 0.0 0.0" xyz="0.0 0.0 0.0" />
   </joint>
+  <!-- arm top table-->
+<xacro:include filename="$(find manipulator_description)/urdf/table.urdf.xacro" />
+ <joint name="table_joint" type="fixed">
+    <parent link="table_top_link" />
+    <child link = "base_link" />
+    <origin xyz="${table_x} ${table_y} ${table_z+table_height}" rpy="0.0 0.1 0.0" />
+  </joint>
   <xacro:ur5_robot prefix="" joint_limited="true"/>
-  <!-- gripper -->
+<!-- gripper -->
   <xacro:include filename="$(find robotiq_arg2f_model_visualization)/urdf/robotiq_arg2f_140_model_macro.xacro" />
   <xacro:robotiq_arg2f_140 prefix=""/>

Commit message: some fixes to urdf and limit the joints in launch

File: urdf/ur5_robotiq_joint_limited_robot.urdf.xacro (robot description, xacro)
@@ -5,17 +5,18 @@
 <!-- ur5 -->
 <xacro:include filename="$(find ur_description)/urdf/ur5.urdf.xacro" />
+<!-- table -->
+<xacro:include filename="$(find manipulator_description)/urdf/table.urdf.xacro" />
  <!-- table leg  to world-->
-  <!--link name="world" /-->
-  <!--joint name="world_joint" type="fixed">
+  <link name="world" />
+  <joint name="world_joint" type="fixed">
     <parent link="world" />
-    <child link = "table_top_link" />
-    <origin rpy="0.0 0.0 0.0" xyz="0.0 0.0 0.0" />
-  </joint-->
+    <child link = "base_link" />
+    <origin xyz="0.0 0.0 0.0" rpy="0.0 0.0 0.0" />
+  </joint>
   <!-- arm top table-->
-<xacro:include filename="$(find manipulator_description)/urdf/table.urdf.xacro" />
  <joint name="table_joint" type="fixed">
-    <parent link="table_top_link" />
-    <child link = "base_link" />
-    <origin xyz="${table_x} -0.21 ${table_height+0.005}" rpy="0.0 0.0 0.0" />
+    <parent link="world"/>
+    <child link="table_top_link" />
+    <origin xyz="-${table_x} +0.21 -${table_height}" rpy="0.0 0.0 0.0" />
   </joint>
   <xacro:ur5_robot prefix="" joint_limited="true"/>
